Commit message: Publish SNS-3DQR demo

File: SNS-3DQR/robots/microduck/robot.urdf (robot description, URDF)
Before this commit: robot microduck, 15 links, 14 joints
Joints:
- joint head_pitch: origin xyz=0 -0.05 -0 rpy=3.1415927 0 0 -> xyz=0 -0.05 -0 rpy=-3.1415927 0 -0
- joint head_roll: origin xyz=-0.0179 0 0.0145 rpy=3.1415927 -1.5707963 3.1415927 -> xyz=-0.0179 0 0.0145 rpy=0 -1.5707963 0
- joint head_yaw: origin xyz=-0 0.0186931 -0.0145 rpy=1.5707969 0 -3.1415927 -> xyz=-0 0.0186931 -0.0145 rpy=-1.5707963 -0 -3.1415927
- joint left_ankle: origin xyz=0 0.042 -0.026 rpy=3.1415927 -0 0 -> xyz=0 0.042 -0.026 rpy=3.1415927 0 0
- joint left_hip_pitch: origin xyz=0.025 0 -0.0185 rpy=-1.5707963 0 -1.5707963 -> xyz=0.025 0 -0.0185 rpy=0 1.5707963 -1.5707963
- joint left_hip_roll: origin xyz=0 0.0165 0.0125 rpy=-1.5707969 -0 0 -> xyz=0 0.0165 0.0125 rpy=-1.5707963 0 -0
- joint left_hip_yaw: origin xyz=0.006 0.0175 -0.005 rpy=3.1415927 -0 1.5707969 -> xyz=0.006 0.0175 -0.005 rpy=-3.1415927 0 -1.5707963
- joint left_knee: origin xyz=0.022 0.0357771 -0.004 rpy=3.1415927 0 1.5707969 -> xyz=0.022 0.0357771 -0.004 rpy=-3.1415927 0 -1.5707963
- joint neck_pitch: origin xyz=0.026 0.0145 0.0324215 rpy=-1.5707969 0 3.1415927 -> xyz=0.026 0.0145 0.0324215 rpy=1.5707963 0 -3.1415927
- joint right_ankle: origin xyz=-0.042 0 -0.026 rpy=-3.1415927 0 1.5707969 -> xyz=-0.042 0 -0.026 rpy=-3.1415927 -0 -1.5707963
- joint right_hip_pitch: origin xyz=0.025 0 -0.0185 rpy=-1.5707963 0 -1.5707963 -> xyz=0.025 0 -0.0185 rpy=0 1.5707963 -1.5707963
- joint right_hip_roll: origin xyz=-0 0.0165 0.0125 rpy=1.5707969 0 3.1415927 -> xyz=-0 0.0165 0.0125 rpy=-1.5707963 0 3.1415927
- joint right_hip_yaw: origin xyz=0.006 -0.0175 -0.005 rpy=3.1415927 0 1.5707969 -> xyz=0.006 -0.0175 -0.005 rpy=-3.1415927 0 -1.5707963
- joint right_knee: origin xyz=-0.022 0.0357771 -0.004 rpy=3.1415927 0 -0 -> xyz=-0.022 0.0357771 -0.004 rpy=-3.1415927 -0 -0

File: SNS-3DQR/robots/triarm/robot.urdf (robot description, URDF)
Before this commit: robot triarm, 18 links, 17 joints
Links:
- link harness_base: geometry visual box size=0.034 0.14 0.014; visual box size=0.034 0.16 0.014
- link harness_yoke: geometry visual box size=0.09 0.04 0.05
Joints:
- joint arm_mount: origin xyz=0.11 0.02 0 rpy=0 1.5708 0 -> xyz=0.06 0.01 0 rpy=0 1.5708 0
- joint harness_yoke_fixed: origin xyz=0.02 0.06 0.18 rpy=0 0 0 -> xyz=0.2 0.03 0.35 rpy=0 0 -0.35

Commit message: Refresh SNS-3DQR demo

File: SNS-3DQR/robots/microduck/robot.urdf (robot description, URDF)
Before this commit: robot microduck, 15 links, 14 joints
Joints:
- joint head_pitch: origin xyz=0 -0.05 -0 rpy=-3.1415927 0 -0 -> xyz=0 -0.05 -0 rpy=3.1415927 -0 0
- joint head_roll: origin xyz=-0.0179 0 0.0145 rpy=0 -1.5707963 0 -> xyz=-0.0179 0 0.0145 rpy=-0 -1.5707963 0
- joint head_yaw: origin xyz=-0 0.0186931 -0.0145 rpy=-1.5707963 -0 -3.1415927 -> xyz=-0 0.0186931 -0.0145 rpy=1.5707963 -0 -3.1415927
- joint left_ankle: origin xyz=0 0.042 -0.026 rpy=3.1415927 0 0 -> xyz=0 0.042 -0.026 rpy=3.1415927 -0 0
- joint left_hip_pitch: origin xyz=0.025 0 -0.0185 rpy=0 1.5707963 -1.5707963 -> xyz=0.025 0 -0.0185 rpy=-1.5707963 -0 -1.5707963
- joint left_hip_roll: origin xyz=0 0.0165 0.0125 rpy=-1.5707963 0 -0 -> xyz=0 0.0165 0.0125 rpy=-1.5707963 -0 0
- joint left_hip_yaw: origin xyz=0.006 0.0175 -0.005 rpy=-3.1415927 0 -1.5707963 -> xyz=0.006 0.0175 -0.005 rpy=3.1415927 -0 1.5707963
- joint left_knee: origin xyz=0.022 0.0357771 -0.004 rpy=-3.1415927 0 -1.5707963 -> xyz=0.022 0.0357771 -0.004 rpy=3.1415927 -0 1.5707963
- joint neck_pitch: origin xyz=0.026 0.0145 0.0324215 rpy=1.5707963 0 -3.1415927 -> xyz=0.026 0.0145 0.0324215 rpy=-1.5707963 0 3.1415927
- joint right_ankle: origin xyz=-0.042 0 -0.026 rpy=-3.1415927 -0 -1.5707963 -> xyz=-0.042 0 -0.026 rpy=-3.1415927 -0 1.5707963
- joint right_hip_pitch: origin xyz=0.025 0 -0.0185 rpy=0 1.5707963 -1.5707963 -> xyz=0.025 0 -0.0185 rpy=-1.5707963 -0 -1.5707963
- joint right_hip_roll: origin xyz=-0 0.0165 0.0125 rpy=-1.5707963 0 3.1415927 -> xyz=-0 0.0165 0.0125 rpy=1.5707963 0 3.1415927
- joint right_hip_yaw: origin xyz=0.006 -0.0175 -0.005 rpy=-3.1415927 0 -1.5707963 -> xyz=0.006 -0.0175 -0.005 rpy=3.1415927 -0 1.5707963
- joint right_knee: origin xyz=-0.022 0.0357771 -0.004 rpy=-3.1415927 -0 -0 -> xyz=-0.022 0.0357771 -0.004 rpy=3.1415927 -0 -0
